File: NRFBlueSlime-Tracker.kicad_sch (KiCad schematic)
At the start: 29 parts, among them J1 532610271, J2 Conn_01x06_Pin, SW1 TS-1088-AR02016, U1 ISP1507-AX-ST, U2 ICM-42688-P, U3 LIS2MDL, U4 ME6211C33R5G, U5 SRV05-4, X1 S2D32.768KB20F30T

Commit message: mdbt42
Parts:
- removed J2: Conn_01x06_Pin, Connector_PinHeader_2.54mm:PinHeader_1x06_P2.54mm_Vertical, symbol Connector:Conn_01x06_Pin
- removed U1: ISP1507-AX-ST, ISP1507AXST, symbol ISP1507-AX-ST:ISP1507-AX-ST
- removed U4: ME6211C33R5G, nrfslime:SOT-353_L2.1-W1.3-P0.65-LS2.3-BL, symbol nrfslime:ME6211C33R5G
- added J2, J3, J4, J5, J6, J7: Conn_01x01, TestPoint:TestPoint_Pad_4.0x4.0mm, symbol Connector_Generic:Conn_01x01
- added U1: MDBT42-512KV2, MDBT42:MDBT42, symbol MDBT42-512KV2:MDBT42
- added U4: RT9080-33GJ5, RT9080:TSOT-23-5_RIT, symbol RT9080:RT9080-33GJ5
Connections:
- net +3V3: now also U1.15 (VDD), U4.5 (VOUT)
- net +BATT: now also J2.1 (Pin_1), U4.1 (VIN), U4.3 (EN)
- net ADC_EN: now also U1.24 (P0.02)
- net BATLVL: now also U1.23 (P0.03)
- net DOCK: now also J7.1 (Pin_1), U1.16 (P0.08)
- net GND: now also J6.1 (Pin_1), U1.1 (GND), U1.14 (GND), U1.25 (GND), U1.37 (GND), U4.2 (GND)
- net INT: now also U1.34 (P0.11)
- net KEY: now also U1.17 (P0.06)
- net LED: now also U1.30 (P0.25)
- net RST: now also J5.1 (Pin_1), U1.6 (P0.21/RESET)
- net SCL: now also U1.2 (P0.23)
- net SDA: now also U1.36 (P0.19)
- net SWC: now also J4.1 (Pin_1), U1.4 (SWDCLK)
- net SWD: now also J3.1 (Pin_1), U1.5 (SWDIO)
- no-connect marks 15 -> 5
Other:
- note added: "Connectors"
- note added: "IMU and Oscillator"
- note added: "LDO"
- note added: "Magnetometer"
- note added: "NRF52832"
- note added: "Programmable Key"
- note added: "Pullups, LED, Battery Sense"
- note added: "TVS"
- moved on the sheet: C10, C11, C6, C7, C8, C9, J1, R1, SW1, U5, X1
