File: NRFBlueSlime-Tracker.kicad_sch (KiCad schematic)
At the start: 60 parts, among them J1 GT-USB-7010ASV, J2 532610271, Q1 AO3401A, SW1 TS-1088-AR02016, U1 ICM-45686, U2 E73-2G4M08S1C, U3 LIS2MDL, U4 EA8103T5R, U5 TP4057-42-SOT26-R, X1 S2D32.768KB20F30T, Y1 Q13FC13500004

Commit message: redo pcb
Parts:
- removed J2: 532610271, Connector_Molex:Molex_PicoBlade_53261-0271_1x02-1MP_P1.25mm_Horizontal, symbol Connector_Generic_MountingPin:Conn_01x02_MountingPin
- added TP7, TP8: TestPoint, TestPoint:TestPoint_Pad_1.0x1.0mm, symbol Connector:TestPoint
- C16, C17: footprint Capacitor_SMD:C_0603_1608Metric -> Capacitor_SMD:C_0402_1005Metric
- C7, C9: footprint Capacitor_SMD:C_0402_1005Metric -> Capacitor_SMD:C_0603_1608Metric
- L1: footprint nrfslime:IND-SMD_L3.0-W3.0 -> Inductor_SMD:L_1210_3225Metric
- LED1: value NCD0402B1 -> XL-1608UBC-04; footprint LED_SMD:LED_0402_1005Metric -> LED_SMD:LED_0603_1608Metric
- LED2: value NCD0402R1 -> XL-1608SURC-06; footprint LED_SMD:LED_0402_1005Metric -> LED_SMD:LED_0603_1608Metric
- LED3: value NCD0402G1 -> XL-1608UGC-06; footprint LED_SMD:LED_0402_1005Metric -> LED_SMD:LED_0603_1608Metric
- Q1: value AO3401A -> NTS2101PT1G; footprint Package_TO_SOT_SMD:SOT-23 -> Package_TO_SOT_SMD:SOT-323_SC-70; symbol Transistor_FET:AO3401A -> Transistor_FET:Q_PMOS_GSD
- R1, R13, R14, R2, R3, R4, R6, R7: footprint Resistor_SMD:R_0603_1608Metric -> Resistor_SMD:R_0402_1005Metric
- R10, R11, R8: footprint Resistor_SMD:R_0402_1005Metric -> Resistor_SMD:R_0603_1608Metric
- U2: footprint nrf:WIRELM-SMD_E73-2G4M08S1C -> nrf:E73-2G4M08S1C_nobottom
- U4: value EA8103T5R -> EA8103DHR; footprint Package_TO_SOT_SMD:SOT-23-5 -> nrfslime:DFN-6_L1.5-W1.5-P0.50-BL-EP1.0; symbol nrfslime:EA8103T5R -> nrfslime:EA8103DHR
- X1: footprint nrfslime:OSC-SMD_4P-L2.5-W2.0-BL -> Crystal:Crystal_SMD_2520-4Pin_2.5x2.0mm
Connections:
- net ADC_EN is gone; now on net ~{ADC_EN}: U2.3 (P0.03)
- net +BATT: now also R10.2, TP7.1; no longer R10.1
- net BATLVL: now also R10.1, R11.2; no longer R10.2, R11.1
- net GND: now also R8.1, U4.4 (GND), U4.7 (EP), TP8.1; no longer R8.2, U4.2 (GND)
- net VBUS: now also R8.2; no longer R8.1
- net VDC: now also U4.2 (EN), U4.6 (VIN); no longer U4.1 (EN), U4.4 (VIN)
- net ~{ADC_EN}: now also R11.1; no longer R11.2
- net at L1.1: now also U4.1 (SW); no longer U4.3 (SW)
- net at R6.2, R7.1: now also U4.3 (FB); no longer U4.5 (FB)
Other:
- moved on the sheet: C14

Commit message: sihashkdasfhjkads
Parts:
- removed D8: 1N5819WS, Diode_SMD:D_SOD-323, symbol Diode:1N5819WS
- removed Q1: NTS2101PT1G, Package_TO_SOT_SMD:SOT-323_SC-70, symbol Transistor_FET:Q_PMOS_GSD
- removed R3, R4: 27, Resistor_SMD:R_0402_1005Metric, symbol Device:R
- removed R9: 1k, Resistor_SMD:R_0402_1005Metric, symbol Device:R
- removed U2: E73-2G4M08S1C, nrf:E73-2G4M08S1C_nobottom, symbol nrf:E73-2G4M08S1C
- removed U5: TP4057-42-SOT26-R, Package_TO_SOT_SMD:SOT-23-6, symbol Battery_Management:TP4057
- added AE1: Antenna_Shield, symbol Device:Antenna_Shield
- added C1, C3: 100p, Capacitor_SMD:C_0402_1005Metric, symbol Device:C
- added C2: 1u, Capacitor_SMD:C_0603_1608Metric, symbol Device:C
- added C4, C5: 15p, Capacitor_SMD:C_0402_1005Metric, symbol Device:C
- added C6: 100n, Capacitor_SMD:C_0402_1005Metric, symbol Device:C
- added C7: 0.8p, Capacitor_SMD:C_0402_1005Metric, symbol Device:C
- added C9: 6.8p, Capacitor_SMD:C_0402_1005Metric, symbol Device:C
- added L1: 4.7n, Inductor_SMD:L_0402_1005Metric, symbol Device:L
- added R1, R2: 27, Resistor_SMD:R_0402_1005Metric, symbol Device:R
- added R11: 10k, Resistor_SMD:R_0402_1005Metric, symbol Device:R
- added U1: nRF52840, Package_DFN_QFN:Nordic_AQFN-73-1EP_7x7mm_P0.5mm, symbol MCU_Nordic:nRF52840
- added U3: BQ24075RGT, Package_DFN_QFN:VQFN-16-1EP_3x3mm_P0.5mm_EP1.6x1.6mm, symbol Battery_Management:BQ24075RGT
- added Y2: XL7EL89CKI-111YLC-32M, Crystal:Crystal_SMD_2016-4Pin_2.0x1.6mm, symbol Device:Crystal_GND24
- C16: renamed from C14; value 1u -> 4.7u
- C17: value 22p -> 4.7u; footprint Capacitor_SMD:C_0402_1005Metric -> Capacitor_SMD:C_0603_1608Metric
- C8: renamed from C16; value 22p -> 6.8p
- R8: value 100k -> 10k; footprint Resistor_SMD:R_0603_1608Metric -> Resistor_SMD:R_0402_1005Metric
- Y1: value Q13FC13500004 -> XKXGI-SUA-32.768K
- renumbered C7 to C10, C8 to C11, C9 to C12, C10 to C13, C12 to C14, C13 to C15, C15 to C18, C3 to C19, C1 to C20, C2 to C21, C4 to C22, C5 to C23, C6 to C24, C11 to C25, D7 to D6, D6 to D7, L1 to L2, R11 to R10, R5 to R3, R1 to R4, R2 to R5, R10 to R9, U4 to U2, U1 to U4, U3 to U5
Connections:
- net +3V3: now also U1.A22 (VDD), U1.AD14 (VDD), U1.AD23 (VDD), U1.B1 (VDD), U1.W1 (VDD), U1.Y2 (VDDH)
- net +BATT: now also C18.2, U3.2 (BAT), U3.3 (BAT); no longer C18.1
- net BATLVL: now also U1.A12 (AIN0/P0.02), U1.AC13 (P0.18/~{RESET})
- net DN: now also R1.1
- net DOCK: now also U1.A20 (P1.10)
- net DP: now also R2.1
- net GND: now also C17.1, C18.1, R12.2, C1.1, C2.1, C3.1, C6.1, C7.1, R11.2, U1.B7 (VSS), U1.EP (VSS), U1.F23 (VSS_PA), U3.15 (SYSOFF), U3.17 (VSS), U3.4 (~{CE}), U3.5 (EN2), U3.8 (VSS), Y2.2, Y2.4; no longer C18.2, R12.1, R8.1
- net INT: now also U1.AC11 (P0.16)
- net KEY: now also U1.B19 (P1.11)
- net LED: now also U1.A14 (P1.15)
- net MISO: now also U1.AD20 (P0.24)
- net MOSI: now also U1.AC21 (P0.25), U1.AD16 (P0.20)
- net OSC_EN: now also U1.A16 (P1.13)
- net SWC: now also U1.AA24 (SWDCLK)
- net SWD: now also U1.AC24 (SWDIO)
- net VBUS: now also U1.AD2 (VBUS), U3.13 (IN); no longer R8.2
- net VDC: now also R8.2, U3.10 (OUT), U3.11 (OUT), U3.6 (EN1)
- net ~{ADC_EN}: now also U1.B15 (P1.14)
- net ~{CS}_IMU: now also U1.AC9 (P0.14)
- net ~{CS}_MAG: now also U1.AD8 (P0.13)
- net at C8.1: now also Y2.3
- net at C8.2: now also U1.B24 (XC1); no longer Y1.1
- net at C17.2: now also LED2.2 (A), LED3.2 (A), R8.1; no longer Y1.2
- net at LED3.1 (K): now also U3.9 (~{CHG})
- net at LED2.1 (K): now also U3.7 (~{PGOOD})
- new net: C9.1, Y2.1
- new net: C9.2, U1.A23 (XC2)
- new net: C3.2, U1.D23 (DEC3)
- new net: R1.2, U1.AD4 (D-)
- new net: C1.2, C2.2, U1.B5 (DEC4), U1.E24 (DEC6)
- new net: C6.2, U1.C1 (DEC1)
- new net: C7.2, L1.2, U1.H23 (ANT)
- new net: R2.2, U1.AD6 (D+)
- new net: C4.1, U1.D2 (XL1/P0.00)
- new net: C5.1, U1.F2 (XL2/P0.01)
- new net: C4.2, Y1.1
- new net: C5.2, Y1.2
- new net: R12.1, U3.1 (TS)
- new net: R11.1, U3.16 (ISET)
- no-connect marks 3 -> 4
Other:
- moved on the sheet: C10, C11, C12, C13, C14, C15, C16, C18, C19, C20, C21, C22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
